File: kicad_project/BlackPanda.kicad_pcb (KiCad board)
At the start: 2 copper layers, 45.9 x 46.3 mm, 91 parts, among them J1 Conn_01x04_Female, J2 USB_A TE Connectivity 292303-7, P1 USB-C-USB-3.2-rescue_USB_C_Pl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, Q1 DDTA143ECA-7-F P08, Q2 DDTA143ECA-7-F P08, Q3 PDTC114EU, SW1 SW_Push, U1 SIS427EDN-T1-GE3, U10 TJA1042TK-3, U11 TJA1042TK-3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

Commit message: -
Other:
- board text removed: "5V"
Changed lines of the file:
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@@
     (effects (font (size 0.9 0.9) (thickness 0.15)) (justify mirror))
-  )
-  (gr_text "5V" (at 193.35 81.34) (layer "F.SilkS")
-    (effects (font (size 0.3 0.3) (thickness 0.075)))
   )
   (gr_text "BAS40WS 43 " (at 204.47 80.51 90) (layer "F.SilkS")
@@
     (effects (font (size 0.4 0.4) (thickness 0.1)))
   )
-  (gr_text "3.3V" (at 193.5 78.8) (layer "F.SilkS")
-    (effects (font (size 0.3 0.3) (thickness 0.075)))
-  )
   (gr_text "+\n" (at 178.89 96.85) (layer "F.SilkS")

Commit message: -
Parts:
- removed R12: 48.7K, Resistor_SMD:R_0603_1608Metric
- removed R13: 10K, Resistor_SMD:R_0402_1005Metric
- removed U6: TPS2549IRTETQ1, Package_DFN_QFN:WQFN-16-1EP_3x3mm_P0.5mm_EP1.75x1.75mm
- added C17: 47uF, Capacitor_SMD:C_0805_2012Metric, F.Cu at (203.2, 78.0)
- added C34: 0.1uF, Capacitor_SMD:C_0402_1005Metric, F.Cu at (199.7, 76.3)
- added Q4: HY12P03C2, Package_SO:PowerPAK_SO-8_Single, F.Cu at (212.8, 79.9)
- added R9: 10K, Resistor_SMD:R_0402_1005Metric, F.Cu at (195.2, 75.9)
- C8: value 100NF -> 10uF
- R26: value 19.1K -> 10K
- R27: value 10K -> 2.2K
- R4: value 4.64K -> 53.6k
- U1: value SIS427EDN-T1-GE3 -> AP22615AWU-7; footprint BlackPanda:SIS427EDN-T1-GE3 -> Package_TO_SOT_SMD:SOT-23-6
- moved U1 15.0 mm to (197.4, 77.5), turned to -90 degrees
- moved R27 5.87 mm to (196.7, 80.4), turned to 0 degrees
- moved C8 2.55 mm to (199.7, 79.4), turned to -90 degrees
- moved R26 1.40 mm to (195.2, 78.9), turned to -90 degrees
- moved R11 1.38 mm to (189.1, 70.9), turned to 180 degrees
- moved J2 0.49 mm to (209.7, 69.8)
- moved Q3 0.35 mm to (202.6, 80.8)
- moved C33 0.16 mm to (208.7, 102.2)
- moved D2 0.07 mm to (205.0, 80.7)
Connections:
- C8 pad 1: +5V -> GND
- C8 pad 2: GND -> +5V
- J2 pad 5: Net-(J2-Pad5) -> GND
- R14 pad 1: BOOT0 -> Net-(U7-Pad60)
- R20 pad 1: Net-(R20-Pad1) -> USB_D-
- R21 pad 2: Net-(R21-Pad2) -> USB_D+
- R26 pad 1: Net-(R26-Pad1) -> Net-(Q3-Pad3)
- R26 pad 2: GND -> +5V
- R27 pad 1: +5V -> GND
- R27 pad 2: Net-(Q3-Pad3) -> Net-(R27-Pad2)
- R4 pad 1: CS -> FB
- SW1 pad 1: USB_PWR -> Net-(U7-Pad60)
- SW1 pad 2: Net-(J2-Pad5) -> +3V3
- U1 pad 1: 12V_Protected -> USB_PWR
- U1 pad 2: 12V_Protected -> GND
- U1 pad 3: 12V_Protected -> Net-(U1-Pad3)
- U1 pad 4: Net-(D2-Pad2) -> Net-(Q3-Pad3)
- U1 pad 5: +12V -> Net-(R27-Pad2)
- U1 pad 6: +12V -> +5V
- U7 pad 60: BOOT0 -> Net-(U7-Pad60)
Routing:
- net Net-(U7-Pad60): track 0.00 -> 67.4 mm, vias 0 -> 2
- net BOOT0: track 60.0 -> 0.00 mm, vias 2 -> 0
- net Net-(J2-Pad5): track 30.3 -> 0.00 mm
- net +3V3: track 234.7 -> 263.6 mm
- net +5V: track 185.3 -> 163.7 mm, vias 9 -> 8
- net CS: track 19.5 -> 0.00 mm, vias 2 -> 0
- net GND: track 191.4 -> 205.5 mm
- net USB_PWR: track 23.6 -> 14.2 mm, vias 4 -> 3
- net Net-(Q3-Pad3): track 3.19 -> 10.5 mm, vias 0 -> 2
- net USB_D-: track 26.0 -> 32.6 mm
- net USB_D+: track 26.1 -> 32.4 mm
- net +12V: track 36.8 -> 31.1 mm
- net Net-(R21-Pad2): track 2.70 -> 0.00 mm
- net Net-(R20-Pad1): track 2.46 -> 0.00 mm
- net Net-(R27-Pad2): track 0.00 -> 1.86 mm
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
Commit message: -
Parts:
- R27: value 2.2K -> 2.4K
Changed lines of the file:
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@@
   (net 44 "FB")
   (net 45 "Net-(R15-Pad1)")
-  (net 46 "Net-(U1-Pad3)")
+  (net 46 "Net-(R9-Pad2)")
   (net 47 "Net-(R27-Pad2)")
   (net 48 "Net-(R22-Pad1)")
@@
   (net 101 "+3V3")
   (net 102 "Net-(D11-Pad1)")
-  (net 103 "Net-(U7-Pad60)")
+  (net 103 "Net-(R14-Pad1)")
   (footprint "Capacitor_SMD:C_0402_1005Metric" (layer "F.Cu")
     (at 199.7 79.43 -90)
@@
       (net 1 "GND") (pinfunction "GND") (pintype "power_in"))
     (pad "3" smd roundrect (at -1.1375 0.95 270) (size 1.325 0.6) (layers "F.Cu" "F.Paste" "F.Mask") (roundrect_rratio 0.25)
-      (net 46 "Net-(U1-Pad3)") (pinfunction "FLG") (pintype "input"))
+      (net 46 "Net-(R9-Pad2)") (pinfunction "FLG") (pintype "input"))
     (pad "4" smd roundrect (at 1.1375 0.95 270) (size 1.325 0.6) (layers "F.Cu" "F.Paste" "F.Mask") (roundrect_rratio 0.25)
       (net 94 "Net-(Q3-Pad3)") (pinfunction "EN") (pintype "bidirectional"))
@@
       (net 3 "+5V") (pintype "passive"))
     (pad "2" smd roundrect (at 0.51 0 270) (size 0.54 0.64) (layers "F.Cu" "F.Paste" "F.Mask") (roundrect_rratio 0.25)
-      (net 46 "Net-(U1-Pad3)") (pintype "passive"))
+      (net 46 "Net-(R9-Pad2)") (pintype "passive"))
     (model "${KICAD6_3DMODEL_DIR}/Resistor_SMD.3dshapes/R_0402_1005Metric.wrl"
       (offset (xyz 0 0 0))
@@
       (effects (font (size 0.5 0.5) (thickness 0.1)))
     )
-    (fp_text value "2.2K" (at 0 1.17) (layer "F.Fab")
+    (fp_text value "2.4K" (at 0 1.17) (layer "F.Fab")
       (effects (font (size 1 1) (thickness 0.15)))
     )
@@
       (net 89 "unconnected-(U7-Pad59)") (pinfunction "PB7") (pintype "bidirectional+no_connect"))
     (pad "60" smd roundrect (at -1.75 -5.675 270) (size 0.3 1.55) (layers "F.Cu" "F.Paste" "F.Mask") (roundrect_rratio 0.25)
-      (net 103 "Net-(U7-Pad60)") (pinfunction "BOOT0") (pintype "input"))
+      (net 103 "Net-(R14-Pad1)") (pinfunction "BOOT0") (pintype "input"))
     (pad "61" smd roundrect (at -2.25 -5.675 270) (size 0.3 1.55) (layers "F.Cu" "F.Paste" "F.Mask") (roundrect_rratio 0.25)
       (net 90 "CAN3_RX") (pinfunction "PB8") (pintype "bidirectional"))
@@
     (fp_line (start -0.525 -0.27) (end 0.525 -0.27) (layer "F.Fab") (width 0.1))
     (pad "1" smd roundrect (at -0.51 0) (size 0.54 0.64) (layers "F.Cu" "F.Paste" "F.Mask") (roundrect_rratio 0.25)
-      (net 103 "Net-(U7-Pad60)") (pintype "passive"))
+      (net 103 "Net-(R14-Pad1)") (pintype "passive"))
     (pad "2" smd roundrect (at 0.51 0) (size 0.54 0.64) (layers "F.Cu" "F.Paste" "F.Mask") (roundrect_rratio 0.25)
       (net 1 "GND") (pintype "passive"))
@@
     (fp_circle (center 0 0) (end 1 0) (layer "B.Fab") (width 0.1) (fill none))
     (pad "1" smd rect (at 3.1 1.85 270) (size 1.8 1.1) (layers "B.Cu" "B.Paste" "B.Mask")
-      (net 103 "Net-(U7-Pad60)") (pinfunction "1") (pintype "passive"))
+      (net 103 "Net-(R14-Pad1)") (pinfunction "1") (pintype "passive"))
     (pad "1" smd rect (at -3.1 1.85 270) (size 1.8 1.1) (layers "B.Cu" "B.Paste" "B.Mask")
-      (net 103 "Net-(U7-Pad60)") (pinfunction "1") (pintype "passive"))
+      (net 103 "Net-(R14-Pad1)") (pinfunction "1") (pintype "passive"))
     (pad "2" smd rect (at -3.1 -1.85 270) (size 1.8 1.1) (layers "B.Cu" "B.Paste" "B.Mask")
       (net 101 "+3V3") (pinfunction "2") (pintype "passive"))

Commit message: inductor
Parts:
- removed R5: 442K, Resistor_SMD:R_0402_1005Metric
- removed R6: 90.9R, Resistor_SMD:R_0402_1005Metric
- L1: value 470NH -> 27nH
- turned R7 to -90 degrees
Connections:
- R7 pad 1: GND -> Net-(R7-Pad1)
- R7 pad 2: Net-(R7-Pad2) -> GND
- U5 pad 3: Net-(R5-Pad1) -> unconnected-(U5-Pad3)
- U5 pad 4: Net-(R7-Pad2) -> Net-(R7-Pad1)
Routing:
- net Net-(R5-Pad1): track 2.87 -> 0.00 mm
- net Net-(R7-Pad2): track 1.75 -> 0.00 mm
- net Net-(R7-Pad1): track 0.00 -> 1.75 mm
- net GND: track 205.5 -> 204.9 mm

Commit message: ...
Connections:
- J2 pad 5: GND -> unconnected-(J2-Pad5)
Routing:
- net GND: track 204.9 -> 203.8 mm
- net unconnected-(J2-Pad5): track 0.00 -> 1.12 mm
Changed lines of the file:
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@@
   (net 102 "Net-(R14-Pad1)")
   (net 103 "unconnected-(U5-Pad3)")
+  (net 104 "unconnected-(J2-Pad5)")
   (footprint "Capacitor_SMD:C_0402_1005Metric" (layer "F.Cu")
     (at 199.7 79.43 -90)
@@
       (net 1 "GND") (pinfunction "GND") (pintype "power_in"))
     (pad "5" thru_hole circle (at 6.57 -2.7 90) (size 3 3) (drill 2.3) (layers *.Cu *.Mask)
-      (net 1 "GND") (pinfunction "Shield") (pintype "passive"))
+      (net 104 "unconnected-(J2-Pad5)") (pinfunction "Shield") (pintype "passive+no_connect"))
     (pad "5" thru_hole circle (at -6.57 -2.7 90) (size 3 3) (drill 2.3) (layers *.Cu *.Mask)
-      (net 1 "GND") (pinfunction "Shield") (pintype "passive"))
+      (net 104 "unconnected-(J2-Pad5)") (pinfunction "Shield") (pintype "passive+no_connect"))
     (model "${KICAD6_3DMODEL_DIR}/Connector_USB.3dshapes/USB_A_TE_292303-7_Horizontal.wrl"
       (offset (xyz 0 0 0))
@@
   (segment (start 184.35 75.15) (end 185.15 75.95) (width 0.2) (layer "F.Cu") (net 1))
   (segment (start 174.72 90.25) (end 174.72 91.27) (width 0.2) (layer "F.Cu") (net 1))
-  (segment (start 207.03 76.42) (end 207.1823 76.2677) (width 0.2) (layer "F.Cu") (net 1))
   (segment (start 199.35 94.15) (end 199.35 95.6) (width 0.5) (layer "F.Cu") (net 1))
   (segment (start 210.26 83.81) (end 210.71 83.81) (width 0.2) (layer "F.Cu") (net 1))
-  (segment (start 207.1823 63.4323) (end 207.03 63.28) (width 0.2) (layer "F.Cu") (net 1))
   (segment (start 197.56952 77.25952) (end 199.22048 77.25952) (width 0.15) (layer "F.Cu") (net 1))
   (segment (start 175.65 83.82) (end 176.07 84.24) (width 0.2) (layer "F.Cu") (net 1))
@@
   (segment (start 210.71 83.81) (end 211.6 84.7) (width 0.6) (layer "B.Cu") (net 1))
   (segment (start 215.73 87.98) (end 215.73 91.47) (width 0.2) (layer "B.Cu") (net 1))
-  (segment (start 207.52 76.91) (end 207.03 76.42) (width 0.2) (layer "B.Cu") (net 1))
   (segment (start 205.49 84.84) (end 205.49 84.137914) (width 0.2) (layer "B.Cu") (net 1))
   (segment (start 210.26 92.07) (end 210.26 91.34) (width 0.2) (layer "B.Cu") (net 1))
@@
   (segment (start 187.2 72.639259) (end 187.2 77.9) (width 0.2) (layer "B.Cu") (net 102))
   (segment (start 183.948 67.985) (end 183.9475 67.985) (width 0.2) (layer "F.Cu") (net 103))
+  (segment (start 207.03 76.42) (end 207.1823 76.2677) (width 0.2) (layer "F.Cu") (net 104))
+  (segment (start 207.1823 63.4323) (end 207.03 63.28) (width 0.2) (layer "F.Cu") (net 104))
+  (segment (start 207.52 76.91) (end 207.03 76.42) (width 0.2) (layer "B.Cu") (net 104))
   (zone (net 0) (net_name "") (layer "F.Cu") (hatch edge 0.508)
     (connect_pads (clearance 0))

Commit message: ...
Parts:
- C15: value 100NF -> 10NF
Changed lines of the file:
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@@
       (effects (font (size 0.5 0.5) (thickness 0.1)))
     )
-    (fp_text value "100NF" (at 0 1.16 90) (layer "F.Fab")
+    (fp_text value "10NF" (at 0 1.16 90) (layer "F.Fab")
       (effects (font (size 1 1) (thickness 0.15)))
     )
